Commit message: Corrections in process_image.cpp

File: Project2/my_robot/urdf/my_robot.xacro (robot description, xacro)
@@ -70,5 +70,5 @@
       <origin xyz="0 0 0" rpy=" 0 1.5707 1.5707"/>
       <geometry>
-        <cylinder length="0.1" radius="0.12"/>
+        <cylinder length="0.1" radius="0.1"/>
       </geometry>
     </collision>
@@ -85,5 +85,5 @@
       <origin xyz="0 0 0" rpy=" 0 1.5707 1.5707"/>
       <geometry>
-        <cylinder length="0.1" radius="0.12"/>
+        <cylinder length="0.1" radius="0.1"/>
       </geometry>
       <material name="red"/>
@@ -94,5 +94,5 @@
       <origin xyz="0 0 0" rpy=" 0 1.5707 1.5707"/>
       <geometry>
-        <cylinder length="0.1" radius="0.12"/>
+        <cylinder length="0.1" radius="0.1"/>
       </geometry>
     </collision>
@@ -109,5 +109,5 @@
       <origin xyz="0 0 0" rpy=" 0 1.5707 1.5707"/>
       <geometry>
-        <cylinder length="0.1" radius="0.12"/>
+        <cylinder length="0.1" radius="0.1"/>
       </geometry>
       <material name="red"/>
